Commit message: changed frame name

File: rpi_robot_description/src/description/rpi_robot_description.urdf (robot description, URDF)
Before this commit: robot rpi_robot, 3 links, 2 joints
Links:
- removed link base_link
Joints:
- joint base_joint: parent base_link -> base_footprint
- joint caster_joint: parent base_link -> base_footprint

Commit message: frame id test

File: rpi_robot_description/src/description/rpi_robot_description.urdf (robot description, URDF)
Before this commit: robot rpi_robot, 2 links, 2 joints
Links:
- removed link base_footprint
- added link base_link
Joints:
- joint base_joint: child base_footprint -> base_link; parent base_footprint -> base_link
- joint caster_joint: parent base_footprint -> base_link
